File: V1.0/WatchDog.kicad_sch (KiCad schematic)
At the start: 10 parts, among them J1 input, J2 output, Q1 NMOS, U1 CN312

Commit message: feat: 更新 WatchDog PCB、原理圖及 Kicad 專案檔案
Changed lines of the file:
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@@
 		)
 		(property "Value" "Earth"
-			(at 106.68 107.95 0)
+			(at 106.68 106.68 0)
 			(show_name no)
 			(do_not_autoplace no)
